Commit message: testing depth camera in gazebo

File: add_post_pro/add_post_pro_robot/urdf/simple_depth_camera.urdf.xacro (robot description, xacro)
@@ -1,4 +1,4 @@
 <?xml version="1.0" encoding="UTF-8"?>
-<robot name="tool" xmlns:xacro="http://www.ros.org/wiki/xacro">
+<robot name="standalone_camera" xmlns:xacro="http://www.ros.org/wiki/xacro">
 	<joint name="J6_to_camera_joint" type="fixed">
     <parent link="J6"/>
@@ -15,5 +15,5 @@
     <origin xyz="0 0 0" rpy="0 0 0"/>
     <geometry>
-        <box size="0.05 0.05 0.05"/> <!-- Size of the box representing the camera; adjust as needed -->
+        <box size="0.5 0.5 0.5"/> <!-- Size of the box representing the camera; adjust as needed -->
     </geometry>
     <material name="blue"> <!-- Simple color material, adjust as needed -->
