Commit message: added depth processing basic functions and testing objects such depth camera

File: add_post_pro/add_post_pro_robot/urdf/camera_robot.xacro (robot description, xacro)
@@ -1,24 +1,24 @@
 <?xml version="1.0"?>
-<robot name="my_robot" xmlns:xacro="http://www.ros.org/wiki/xacro">
+<robot xmlns:xacro="http://www.ros.org/wiki/xacro">
   <!-- Properties -->
   <xacro:property name="camera_width" value="0.05"/>
   <xacro:property name="camera_height" value="0.03"/>
   <xacro:property name="camera_depth" value="0.05"/>
-  <!-- World Link Definition -->
-  <link name="world"/>
-  <!-- Base Link Definition -->
-  <link name="base_link">
-    <inertial>
-      <origin xyz="0 0 0" rpy="0 0 0"/>
-      <mass value="0.001"/>
-      <inertia ixx="1.0e-6" ixy="0" ixz="0" iyy="1.0e-6" iyz="0" izz="1.0e-6"/>
-    </inertial>
-  </link>
-  <!-- Joint connecting World to Base Link -->
-  <joint name="joint_w" type="fixed">
-    <parent link="world"/>
-    <child link="base_link"/>
-    <origin xyz="0 0 0"/>
-  </joint>
+    <!-- World Link Definition -->
+    <link name="world"/>
+    <!-- Base Link Definition -->
+    <link name="base_link">
+        <inertial>
+            <origin xyz="0 0 0" rpy="0 0 0"/>
+            <mass value="0.001"/>
+            <inertia ixx="1.0e-6" ixy="0" ixz="0" iyy="1.0e-6" iyz="0" izz="1.0e-6"/>
+        </inertial>
+    </link>
+    <!-- Joint connecting World to Base Link -->
+    <joint name="joint_w" type="fixed">
+        <parent link="world"/>
+        <child link="base_link"/>
+        <origin xyz="0 0 0"/>
+    </joint>
   <link name="camera_link">
     <visual>
@@ -40,12 +40,13 @@
     </inertial>
   </link>
-  <joint name="base_to_camera_joint" type="fixed">
+ <joint name="base_to_camera_joint" type="fixed">
     <parent link="base_link"/>
     <child link="camera_link"/>
-    <origin xyz="1 0 0.5" rpy="0 0 0"/>
-  </joint>
-  <!-- Depth Camera Plugin -->
+    <origin xyz="0 0 0.5" rpy="0 0 0"/> <!-- This positions the camera 1 unit higher relative to the base_link -->
+ </joint>
+  <!-- Camera Link -->
+  <!-- Camera Plugin -->
   <gazebo reference="camera_link">
-    <sensor type="depth" name="depth_camera_sensor">
+    <sensor type="camera" name="camera_sensor">
       <update_rate>30.0</update_rate>
       <camera>
@@ -54,5 +55,4 @@
           <width>640</width>
           <height>480</height>
-          <format>R8G8B8</format>
         </image>
         <clip>
@@ -61,10 +61,10 @@
         </clip>
       </camera>
-      <plugin name="depth_camera_controller" filename="libgazebo_ros_depth_camera.so">
+      <plugin name="camera_controller" filename="libgazebo_ros_camera.so">
         <alwaysOn>true</alwaysOn>
         <updateRate>0.0</updateRate>
-        <cameraName>robot/depth_camera</cameraName>
-        <imageTopicName>depth_image_raw</imageTopicName>
-        <cameraInfoTopicName>depth_camera_info</cameraInfoTopicName>
+        <cameraName>robot/camera</cameraName>
+        <imageTopicName>image_raw</imageTopicName>
+        <cameraInfoTopicName>camera_info</cameraInfoTopicName>
         <frameName>camera_link</frameName>
       </plugin>

File: add_post_pro/add_post_pro_robot/urdf/free_depth_camera.urdf.xacro (robot description, xacro)
@@ -5,21 +5,15 @@
   <xacro:property name="camera_height" value="0.03"/>
   <xacro:property name="camera_depth" value="0.05"/>
-  <!-- World Link Definition -->
+  <!-- Define the world link -->
   <link name="world"/>
-  <!-- Base Link Definition -->
-  <link name="base_link">
-    <inertial>
-      <origin xyz="0 0 0" rpy="0 0 0"/>
-      <mass value="0.001"/>
-      <inertia ixx="1.0e-6" ixy="0" ixz="0" iyy="1.0e-6" iyz="0" izz="1.0e-6"/>
-    </inertial>
-  </link>
-  <!-- Joint connecting World to Base Link -->
-  <joint name="joint_w" type="fixed">
+  <!-- Joint to keep the cube floating -->
+  <joint name="floating_joint" type="fixed">
     <parent link="world"/>
-    <child link="base_link"/>
-    <origin xyz="0 0 0"/>
+    <child link="camera_link"/>
+    <origin xyz="0 2 1" rpy="0 0 0"/>
   </joint>
+  <!-- Camera Link Definition -->
   <link name="camera_link">
+    <gravity>0 </gravity>
     <visual>
       <geometry>
@@ -40,9 +34,4 @@
     </inertial>
   </link>
-  <joint name="base_to_camera_joint" type="fixed">
-    <parent link="base_link"/>
-    <child link="camera_link"/>
-    <origin xyz="1 0 0.5" rpy="0 0 0"/>
-  </joint>
   <!-- Depth Camera Plugin -->
   <gazebo reference="camera_link">
