Commit message: Generate a working depth camera in depth_processing that can move freely in space unaffected by gravity

File: add_post_pro/add_post_pro_robot/urdf/free_depth_camera.urdf.xacro (robot description, xacro)
@@ -1,19 +1,18 @@
 <?xml version="1.0"?>
-<robot name="my_robot" xmlns:xacro="http://www.ros.org/wiki/xacro">
+<robot name="camera_robot">
   <!-- Properties -->
-  <xacro:property name="camera_width" value="0.05"/>
-  <xacro:property name="camera_height" value="0.03"/>
-  <xacro:property name="camera_depth" value="0.05"/>
-  <!-- Define the world link -->
-  <link name="world"/>
-  <!-- Joint to keep the cube floating -->
-  <joint name="floating_joint" type="fixed">
+  <property name="camera_width" value="0.05"/>
+  <property name="camera_height" value="0.03"/>
+  <property name="camera_depth" value="0.05"/>
+  <!-- Dummy Link -->
+  <!-- <link name="world"/> -->
+  <!-- Dummy Joint -->
+  <!-- <joint name="world_to_camera_joint" type="fixed">
     <parent link="world"/>
     <child link="camera_link"/>
-    <origin xyz="0 2 1" rpy="0 0 0"/>
-  </joint>
+    <origin xyz="0 0 0" rpy="0 0 0"/>
+  </joint> -->
   <!-- Camera Link Definition -->
   <link name="camera_link">
-    <gravity>0 </gravity>
     <visual>
       <geometry>
@@ -34,6 +33,7 @@
     </inertial>
   </link>
-  <!-- Depth Camera Plugin -->
+  <!-- Gazebo plugins -->
   <gazebo reference="camera_link">
+    <gravity>0</gravity>
     <sensor type="depth" name="depth_camera_sensor">
       <update_rate>30.0</update_rate>
@@ -58,5 +58,21 @@
         <frameName>camera_link</frameName>
       </plugin>
-      <visualize>1</visualize>
+      <visualize>true</visualize>
+    </sensor>
+    <sensor type="camera" name="visualize_camera_sensor">
+      <update_rate>30.0</update_rate>
+      <camera>
+        <horizontal_fov>1.3962634</horizontal_fov>
+        <image>
+          <width>640</width>
+          <height>480</height>
+          <format>R8G8B8</format>
+        </image>
+        <clip>
+          <near>0.01</near>
+          <far>100</far>
+        </clip>
+      </camera>
+      <visualize>true</visualize>
     </sensor>
   </gazebo>
