Commit message: Lab Setup

File: add_post_pro/add_post_pro_robot/urdf/add_post_pro_robot.urdf.xacro (robot description, xacro)
@@ -3,9 +3,9 @@
     <xacro:arg name="sim" default="True" />
     <xacro:include filename="$(find denso_robot_descriptions)/vs6577_description/urdf/vs6577.urdf.xacro"/>
-    <!-- <xacro:include filename="$(find add_post_pro_robot)/urdf/turntable.urdf.xacro"/> -->
+    <xacro:include filename="$(find add_post_pro_robot)/urdf/turntable.urdf.xacro"/>
     <!-- Create camera instance -->
-    <!-- <turntable parent="world">
+    <turntable parent="world">
 		<origin xyz="0 -.6 0.16" rpy="0 0 0"/>
-    </turntable> -->
+    </turntable>
     <xacro:include filename="$(find add_post_pro_robot)/urdf/multisensor_holder.urdf.xacro"/>
 </robot>

File: add_post_pro/add_post_pro_robot/urdf/multisensor_holder.urdf.xacro (robot description, xacro)
@@ -26,5 +26,5 @@
 			<origin rpy="0 0 0" xyz="0 0 0"/>
 			<geometry>
-				<mesh filename="package://add_post_pro_robot/meshes/better_holder.stl" scale=".001 .001 .001"/>
+				<mesh filename="package://add_post_pro_robot/meshes/multisensor_holder_origin.stl" scale=".001 .001 .001"/>
 			</geometry>
 		</visual>
@@ -32,5 +32,5 @@
 			<origin rpy="0 0 0" xyz="0 0 0"/>
 			<geometry>
-				<mesh filename="package://add_post_pro_robot/meshes/better_holder.stl" scale=".001 .001 .001"/>
+				<mesh filename="package://add_post_pro_robot/meshes/multisensor_holder_origin.stl" scale=".001 .001 .001"/>
 			</geometry>
 		</collision>
@@ -48,9 +48,11 @@
 		<origin rpy="0.000000 0.000000 0.000000" xyz="0.000000 0.000000 0.000000"/>
 	</joint>
+	<!--Changes here!-->
 	<joint name="end_effector_magnet" type="fixed">
 		<parent link="J6"/>
 		<child link="EEF_sensor_holder"/>
-		<origin rpy="0.000000 0.000000 ${M_PI}" xyz="0.000000 0.000000 0.000000"/>
+		<origin rpy="0.000000 0.00000 ${225*M_PI/180}" xyz="0.000000 0.000000 0.000000"/>
 	</joint>
+	<!--Changes here!-->
     <joint name="end_effector_scanner_holder" type="fixed">
     	<parent link="EEF_sensor_holder"/>

File: add_post_pro/add_post_pro_robot/urdf/scancontrol.xacro (robot description, xacro)
@@ -1,4 +1,5 @@
 <?xml version="1.0" encoding="UTF-8"?>
 <robot xmlns:xacro="http://www.ros.org/wiki/xacro">
+<xacro:property name="M_PI" value="3.1415926535897931" />
 <xacro:macro name="scancontrol2900-100" params="parent">
 <!-- DONE -->
@@ -24,19 +25,19 @@
 	</link>
     <link name="scancontrol2900-50_laser"/>
-    <link name="true_laser" />
+    <link name = "true_laser"/>
     <joint name="end_effector_scanner" type="fixed">
     	<parent link="${parent}"/>
 		<child link="EEF_scancontrol"/>
-		<origin rpy="0.000000 0.000000 0.000000" xyz="0.000000 0.000000 0.000000"/>
+		<origin rpy="0.000000 0.0000 ${M_PI}" xyz="0.000000 0.000000 0.000000"/>
     </joint>
     <joint name="laser_joint" type="fixed">
         <parent link="EEF_scancontrol" />
         <child link="scancontrol2900-50_laser" />
-        <origin xyz="0 -0.0324522 -.0761366" rpy="0 ${M_PI/2} ${-M_PI/2}"/>
+        <origin xyz="0 -0.0324522 -.0761366" rpy="0 0 ${M_PI}"/>
     </joint>
     <joint name="imaginary_joint" type="fixed">
         <parent link="scancontrol2900-50_laser" />
         <child link="true_laser" />
-        <origin xyz="0 0 0" rpy="0 ${M_PI/2} 0"/>
+        <origin xyz="0 0 0" rpy="0 0 ${M_PI/2}"/>
     </joint>
         <!-- <origin xyz="0 -0.0324522 -.0761366" rpy="${M_PI} ${M_PI/2} ${M_PI/2}"/> -->

File: add_post_pro/add_post_pro_robot/urdf/tool_holder.urdf.xacro (robot description, xacro)
@@ -1,3 +1,2 @@
-<?xml version="1.0" encoding="UTF-8"?>
 <robot name="tool" xmlns:xacro="http://www.ros.org/wiki/xacro">
 	<!-- DONE -->

File: add_post_pro/add_post_pro_robot/urdf/turntable.urdf.xacro (robot description, xacro)
@@ -56,5 +56,4 @@
             <!-- <limit effort="1000.0" lower="-6.28" upper="6.28" velocity="0.5"/> -->
             <limit effort="1000.0" velocity="0.5" />
-            <limit effort="1000.0"  />
             <axis xyz="0 0 1" />
         </joint>

File: add_post_pro/denso_robot_ros/denso_robot_descriptions/vs6577_description/urdf/vs6577.urdf.xacro (robot description, xacro)
@@ -16,5 +16,5 @@
 	<link name="base_link">
 		<visual>
-			<origin rpy="0 0 0" xyz="0 0.0 0"/>
+			<origin rpy="0 0 0" xyz="0 0 0"/>
 			<geometry>
 				<mesh filename="package://denso_robot_descriptions/vs6577_description/meshes/base_link.dae" scale="1 1 1"/>
@@ -22,5 +22,5 @@
 		</visual>
 		<collision>
-			<origin rpy="0 0 0" xyz="0 0.0 0"/>
+			<origin rpy="0 0 0" xyz="0 0 0"/>
 			<geometry>
 				<mesh filename="package://denso_robot_descriptions/vs6577_description/meshes/base_link.dae" scale="1 1 1"/>
@@ -29,5 +29,5 @@
 		<inertial>
 			<mass value="1"/>
-			<origin rpy="0.000000 0.000000 0.000000" xyz="0.000000 0.0 0.000000"/>
+			<origin rpy="0.000000 0.000000 0.000000" xyz="0.000000 0.000000 0.000000"/>
 			<inertia ixx="1" ixy="0" ixz="0" iyy="1" iyz="0" izz="1"/>
 		</inertial>
@@ -177,5 +177,5 @@
 		<parent link="base_link"/>
 		<child link="J1"/>
-		<origin rpy="0.000000 0.000000 0.000000" xyz="0.000000 0.0 0.000000"/>
+		<origin rpy="0.000000 0.000000 0.000000" xyz="0.000000 0.000000 0.000000"/>
 		<axis xyz="-0.000000 -0.000000 1.000000"/>
 		<limit effort="100" lower="-2.96706" upper="2.96706" velocity="1"/>
@@ -203,6 +203,5 @@
 		<origin rpy="0.000000 0.000000 0.000000" xyz="-0.090000 0.000000 -0.700000"/>
 		<axis xyz="-0.000000 -0.000000 1.000000"/>
-		<!-- <limit effort="100" lower="-3.316126" upper="3.316126" velocity="1"/> -->
-		<limit effort="100" lower="-3.14159" upper="3.14159" velocity="1"/>
+		<limit effort="100" lower="-3.316126" upper="3.316126" velocity="1"/>
 		<dynamics damping="0" friction="0"/>
 	</joint>
@@ -220,6 +219,5 @@
 		<origin rpy="0.000000 0.000000 0.000000" xyz="0.000000 0.000000 0.080000"/>
 		<axis xyz="-0.000000 -0.000000 1.000000"/>
-		<!-- <limit effort="100" lower="-6.283185" upper="6.283185" velocity="1"/> -->
-		<limit effort="100" lower="-3.14159" upper="3.14159" velocity="1"/>
+		<limit effort="100" lower="-6.283185" upper="6.283185" velocity="1"/>
 		<dynamics damping="0" friction="0"/>
 	</joint>
