Commit message: laser scanner updates

File: add_post_pro/add_post_pro_robot/urdf/add_post_pro_robot_b120.urdf.xacro (robot description, xacro)
@@ -3,3 +3,4 @@
     <xacro:include filename="$(find denso_robot_descriptions)/vs6577_description/urdf/vs6577.urdf.xacro"/>
     <xacro:include filename="$(find add_post_pro_robot)/urdf/multisensor_holder.urdf.xacro"/>
+    <!-- <xacro:include filename="$(find add_post_pro_robot)/urdf/l515_mount.urdf.xacro"/> -->
 </robot>

File: add_post_pro/add_post_pro_robot/urdf/scancontrol.xacro (robot description, xacro)
@@ -39,5 +39,5 @@
         <parent link="scancontrol2900-50_laser" />
         <child link="true_laser" />
-        <origin xyz="0 0 0" rpy="0 0 ${M_PI/2}"/>
+        <origin xyz="0 0 0" rpy="${M_PI} 0 0"/>
     </joint>
         <!-- <origin xyz="0 -0.0324522 -.0761366" rpy="${M_PI} ${M_PI/2} ${M_PI/2}"/> -->
