Commit message: added heatmap for error visualization of scans vs nominal

File: add_post_pro/add_post_pro_robot/urdf/random_objects.xacro (robot description, xacro)
@@ -29,5 +29,5 @@
   </joint> -->
   <!-- Cube -->
-  <link name="cube_link">
+  <!-- <link name="cube_link">
     <visual>
       <geometry>
@@ -52,5 +52,29 @@
     <child link="cube_link"/>
     <origin xyz="0 0 0.25"/>
-  </joint>
+  </joint> -->
+  <link name="cube_link">
+  <visual>
+    <geometry>
+        <mesh filename="package://depth_processing/saved_models/cube.stl" scale="1.0 1.0 1.0" />
+    </geometry>
+    <material name="default">
+      <color rgba="1 1 1 1"/>
+    </material>
+  </visual>
+  <collision>
+    <geometry>
+        <mesh filename="package://depth_processing/saved_models/cube.stl" scale="1.0 1.0 1.0" />
+    </geometry>
+  </collision>
+  <inertial>
+			<mass value="0.5"/>
+			<inertia ixx="1" ixy="0" ixz="0" iyy="1" iyz="0" izz="1"/>
+		</inertial>
+</link>
+<joint name="root_to_stl_model" type="fixed">
+  <parent link="root_link"/>
+  <child link="cube_link"/>
+  <origin xyz="0 0 0.25"/>
+</joint>
   <!-- Sphere -->
   <!-- <link name="sphere_link">

Commit message: checkpoint, started view planner view_plan.cpp

File: add_post_pro/add_post_pro_robot/urdf/random_objects.xacro (robot description, xacro)
@@ -56,5 +56,5 @@
   <visual>
     <geometry>
-        <mesh filename="package://depth_processing/saved_models/cube.stl" scale="1.0 1.0 1.0" />
+        <mesh filename="package://depth_processing/saved_models/remesh_bell.stl" scale="1.0 1.0 1.0 " />
     </geometry>
     <material name="default">
@@ -64,5 +64,5 @@
   <collision>
     <geometry>
-        <mesh filename="package://depth_processing/saved_models/cube.stl" scale="1.0 1.0 1.0" />
+        <mesh filename="package://depth_processing/saved_models/remesh_bell.stl" scale="1.0 1.0 1.0 " />
     </geometry>
   </collision>
@@ -75,5 +75,5 @@
   <parent link="root_link"/>
   <child link="cube_link"/>
-  <origin xyz="0 0 0.25"/>
+  <origin xyz="0 0 0"/>
 </joint>
   <!-- Sphere -->
