Commit message: Merging Live Bringup and 7DOF script

File: add_post_pro/add_post_pro_robot/urdf/add_post_pro_equiv.urdf.xacro (robot description, xacro)
@@ -10,7 +10,7 @@
     <xacro:include filename="$(find denso_robot_descriptions)/metrology_description/urdf/metrology.urdf.xacro"/>
     <xacro:include filename="$(find add_post_pro_robot)/urdf/turntable_equiv.urdf.xacro"/>
-    <!-- Create camera instance --> -->
-    <turntable parent="world">
-		<origin xyz="0 -${turntable_offset} 0.16" rpy="0 0 0"/>
+    <!-- Create camera instance -->
+    <turntable parent="world" base_height="0.062" plate_height="0.006" plate_radius="0.250">
+        <origin xyz="0 -${turntable_offset} 0.16" rpy="0 0 0"/>
     </turntable>
     <xacro:include filename="$(find add_post_pro_robot)/urdf/multisensor_holder.urdf.xacro"/>

File: add_post_pro/add_post_pro_robot/urdf/turntable_equiv.urdf.xacro (robot description, xacro)
@@ -1,10 +1,10 @@
 <?xml version="1.0" ?>
 <robot xmlns:xacro="http://www.ros.org/wiki/xacro">
-    <xacro:macro name="turntable" params="parent *origin">
+    <xacro:macro name="turntable" params="parent *origin base_height plate_height plate_radius">
         <link name="turntable_base">
             <visual>
                 <origin rpy="0 0 0" xyz="0 0 0" />
                 <geometry>
-                    <cylinder length=".32" radius=".02" />
+                    <cylinder length="${base_height}" radius=".02" />
                 </geometry>
             </visual>
@@ -12,5 +12,5 @@
                 <origin rpy="0 0 0" xyz="0 0 0" />
                 <geometry>
-                    <cylinder length=".32" radius=".02" />
+                    <cylinder length="${base_height}" radius=".02" />
                 </geometry>
             </collision>
@@ -25,8 +25,8 @@
                 <origin rpy="0 0 0" xyz="0 0 0" />
                 <geometry>
-                    <cylinder length=".01" radius=".15" />
+                    <cylinder length="${plate_height}" radius="${plate_radius}" />
                 </geometry>
-                <material name="Red">
-                    <color rgba="1.0 0 0 1.0" />
+                <material name="DarkGray">
+                    <color rgba="0.1 0.1 0.1 1.0" />
                 </material>
             </visual>
@@ -34,5 +34,5 @@
                 <origin rpy="0 0 0" xyz="0 0 0" />
                 <geometry>
-                    <cylinder length=".01" radius=".15" />
+                    <cylinder length="${plate_height}" radius="${plate_radius}" />
                 </geometry>
             </collision>
@@ -48,10 +48,10 @@
             <child link="turntable_base" />
             <!-- <xacro:insert_block name="origin"/> -->
-            <origin rpy="0 0 0" xyz="0 0 0.16" />
+            <origin rpy="0 0 0" xyz="0 0 0${base_height/2}" />
         </joint>
         <joint name="turntable_revolve_joint" type="continuous">
             <parent link="turntable_base" />
             <child link="turntable_plate" />
-            <origin rpy="0.000000 0.000000 0.000000" xyz="0.000000 0.000000 .16" />
+            <origin rpy="0.000000 0.000000 0.000000" xyz="0.000000 0.000000 ${base_height/2}" />
             <!-- <limit effort="1000.0" lower="-6.28" upper="6.28" velocity="0.5"/> -->
             <limit effort="1000.0" velocity="10" />

File: add_post_pro/denso_robot_ros/denso_robot_descriptions/metrology_description/urdf/metrology.urdf.xacro (robot description, xacro)
@@ -33,5 +33,5 @@
 		<visual>
 		<!-- change y here to length /2 -->
-			<origin rpy="0 1.570796 1.570796" xyz="0 ${turntable_offset/2} 0"/>
+			<origin rpy="0 1.570796 1.570796" xyz="0 -${turntable_offset/2} 0"/>
 			<geometry>
 			<!-- change length here -->
@@ -229,5 +229,5 @@
 		<child link="base_link"/>
 		<!-- Here change length -->
-		<origin xyz="0 ${turntable_offset} 0"/>
+		<origin xyz="0 -${turntable_offset} 0"/>
 	</joint>
 	<joint name="joint_1" type="revolute">
