Commit message: Fall2023 batch commit

File: add_post_pro/add_post_pro_robot/urdf/turntable_equiv.urdf.xacro (robot description, xacro)
@@ -55,5 +55,5 @@
             <origin rpy="0.000000 0.000000 0.000000" xyz="0.000000 0.000000 ${base_height/2}" />
             <!-- <limit effort="1000.0" lower="-6.28" upper="6.28" velocity="0.5"/> -->
-            <limit effort="1000.0" velocity="10" />
+            <limit effort="1000.0" velocity="0.5" />
             <axis xyz="0 0 1" />
         </joint>

Commit message: Working Model

File: add_post_pro/add_post_pro_robot/urdf/turntable_equiv.urdf.xacro (robot description, xacro)
@@ -48,5 +48,5 @@
             <child link="turntable_base" />
             <!-- <xacro:insert_block name="origin"/> -->
-            <origin rpy="0 0 0" xyz="0 0 0${base_height/2}" />
+            <origin rpy="0 0 0" xyz="0 0 ${base_height/2}" />
         </joint>
         <joint name="turntable_revolve_joint" type="continuous">
