Commit message: Updates

File: add_post_pro/add_post_pro_simulation/urdf/add_post_pro_robot.urdf.xacro (robot description, xacro)
@@ -297,5 +297,5 @@
             </geometry>
         </collision>
-<inertial>
+        <inertial>
             <origin rpy="0 0 0" xyz="0 0 0" />
             <mass value="1" />
@@ -649,5 +649,5 @@
     <!-- <origin xyz="0 -0.0324522 -.0761366" rpy="${M_PI} ${M_PI/2} ${M_PI/2}"/> -->
     <gazebo reference="scancontrol2900-50_laser">
-        <sensor name="scancontrol" type="gpu_ray">
+        <sensor name="scancontrol" type="ray">
             <pose>0 0 0 0 0 0</pose>
             <visualize>true</visualize>
@@ -668,5 +668,5 @@
                 </range>
             </ray>
-            <plugin filename="libgazebo_ros_gpu_laser.so" name="scancontrol_laser">
+            <plugin filename="libgazebo_ros_laser.so" name="scancontrol_laser">
                 <topicName>/arm/laser_scan</topicName>
                 <frameName>scancontrol2900-50_laser</frameName>
